File: projects/body-cooler/hardware/body-cooler.sch (KiCad schematic (older format))
At the start: 32 parts, among them J1 漏水探针, K1 5V低电平触发, K2 5V低电平触发, K3 5V低电平触发, K4 5V低电平触发, K5 5V低电平触发, M1 365 隔膜泵, SW1 浮子液位(常开), SW2 急停/总电源(常闭), SW3 按键A, SW4 按键B, T1 防水探头1, T2 防水探头2, T3 防水探头3, U1 ESP32-S3-N16R8

Commit message: fix(hardware): 符号引用改用标准「工程库名:符号名」写法，LIBS 行列两个库 —— 修导入后元件不显示
Parts:
- BT1: symbol body-cooler-cache:BATTERY-3S -> body-cooler:BATTERY-3S
- D1: symbol body-cooler-cache:D-SCHOTTKY -> body-cooler:D-SCHOTTKY
- F1: symbol body-cooler-cache:FUSE -> body-cooler:FUSE
- FS1: symbol body-cooler-cache:FLOW-YF-S401 -> body-cooler:FLOW-YF-S401
- J1: symbol body-cooler-cache:CONN-2 -> body-cooler:CONN-2
- K1, K2, K3, K4, K5: symbol body-cooler-cache:RELAY-5V-LOW -> body-cooler:RELAY-5V-LOW
- LS1: symbol body-cooler-cache:BUZZER -> body-cooler:BUZZER
- M1: symbol body-cooler-cache:PUMP-365 -> body-cooler:PUMP-365
- PS1: symbol body-cooler-cache:PWR-MODULE -> body-cooler:PWR-MODULE
- R10, R11, R6, R7, R8, R9, RP1, RP2, RP3, RP4, RP5: symbol body-cooler-cache:R -> body-cooler:R
- SW1: symbol body-cooler-cache:SW-LEVER -> body-cooler:SW-LEVER
- SW2: symbol body-cooler-cache:SW-NC -> body-cooler:SW-NC
- SW3, SW4: symbol body-cooler-cache:SW-PUSH -> body-cooler:SW-PUSH
- T1, T2, T3: symbol body-cooler-cache:DS18B20 -> body-cooler:DS18B20
- U1: symbol body-cooler-cache:ESP32-S3-DEVKITC -> body-cooler:ESP32-S3-DEVKITC
Changed lines of the file:
@@
 EESchema Schematic File Version 4
-LIBS:body-cooler-cache
+LIBS:body-cooler body-cooler-cache
 EELAYER 29 0
 EELAYER END
@@
 【一】12V 电源树
 $Comp
-L body-cooler-cache:BATTERY-3S BT1
+L body-cooler:BATTERY-3S BT1
 U 1 1 5F000001
 P 1500 2300
@@
 $EndComp
 $Comp
-L body-cooler-cache:FUSE F1
+L body-cooler:FUSE F1
 U 1 1 5F000008
 P 2700 1900
@@
 $EndComp
 $Comp
-L body-cooler-cache:PWR-MODULE PS1
+L body-cooler:PWR-MODULE PS1
 U 1 1 5F00000F
 P 5900 2300
@@
 左右两侧都是 500mil 短支线 + 网络标签，靠名字连接
 $Comp
-L body-cooler-cache:ESP32-S3-DEVKITC U1
+L body-cooler:ESP32-S3-DEVKITC U1
 U 1 1 5F000016
 P 6200 5200
@@
 IN 拉低 = 吸合；释放时 GPIO 变高阻，由 10k 上拉到 5V 才彻底截止
 $Comp
-L body-cooler-cache:RELAY-5V-LOW K1
+L body-cooler:RELAY-5V-LOW K1
 U 1 1 5F00001D
 P 10400 1900
@@
 NC 不接
 $Comp
-L body-cooler-cache:RELAY-5V-LOW K2
+L body-cooler:RELAY-5V-LOW K2
 U 1 1 5F000024
 P 10400 3300
@@
 NC 不接
 $Comp
-L body-cooler-cache:RELAY-5V-LOW K3
+L body-cooler:RELAY-5V-LOW K3
 U 1 1 5F00002B
 P 10400 4700
@@
 NC 不接
 $Comp
-L body-cooler-cache:RELAY-5V-LOW K4
+L body-cooler:RELAY-5V-LOW K4
 U 1 1 5F000032
 P 10400 6100
@@
 NC 不接
 $Comp
-L body-cooler-cache:RELAY-5V-LOW K5
+L body-cooler:RELAY-5V-LOW K5
 U 1 1 5F000039
 P 10400 7500
@@
 【四】泵主回路：电池+ -> 保险丝 -> 继电器 COM/NO -> 泵+ -> 泵- -> 电池-
 $Comp
-L body-cooler-cache:PUMP-365 M1
+L body-cooler:PUMP-365 M1
 U 1 1 5F000040
 P 14300 1900
@@
 GND
 $Comp
-L body-cooler-cache:D-SCHOTTKY D1
+L body-cooler:D-SCHOTTKY D1
 U 1 1 5F000047
 P 14300 2700
@@
 ESP32 复位期间 GPIO 是高阻，靠它把 IN 明确拉到 5V，继电器才彻底截止
 $Comp
-L body-cooler-cache:R RP1
+L body-cooler:R RP1
 U 1 1 5F00004E
 P 12300 8800
@@
 K1_IN
 $Comp
-L body-cooler-cache:R RP2
+L body-cooler:R RP2
 U 1 1 5F000055
 P 13300 8800
@@
 K2_IN
 $Comp
-L body-cooler-cache:R RP3
+L body-cooler:R RP3
 U 1 1 5F00005C
 P 14300 8800
@@
 K3_IN
 $Comp
-L body-cooler-cache:R RP4
+L body-cooler:R RP4
 U 1 1 5F000063
 P 15300 8800
@@
 K4_IN
 $Comp
-L body-cooler-cache:R RP5
+L body-cooler:R RP5
 U 1 1 5F00006A
 P 16300 8800
@@
 5.1 DS18B20 单总线温度（4.7k 上拉到 3V3，整条总线只加一只）
 $Comp
-L body-cooler-cache:R R11
+L body-cooler:R R11
 U 1 1 5F000071
 P 1300 9000
@@
 OW_DQ
 $Comp
-L body-cooler-cache:DS18B20 T1
+L body-cooler:DS18B20 T1
 U 1 1 5F000078
 P 3000 8800
@@
 GND
 $Comp
-L body-cooler-cache:DS18B20 T2
+L body-cooler:DS18B20 T2
 U 1 1 5F00007F
 P 3000 9800
@@
 GND
 $Comp
-L body-cooler-cache:DS18B20 T3
+L body-cooler:DS18B20 T3
 U 1 1 5F000086
 P 3000 10800
@@
 5.2 电池电压采样（100k / 18k = 6.556:1，必须走 ADC1）
 $Comp
-L body-cooler-cache:R R6
+L body-cooler:R R6
 U 1 1 5F00008D
 P 5000 9000
@@
 $EndComp
 $Comp
-L body-cooler-cache:R R7
+L body-cooler:R R7
 U 1 1 5F000094
 P 5000 9800
@@
 5.3 水流传感器（5V 方波经 2.2k+10k/20k 分压到 3.11V 进 GPIO10）
 $Comp
-L body-cooler-cache:R R8
+L body-cooler:R R8
 U 1 1 5F00009B
 P 7000 9000
@@
 $EndComp
 $Comp
-L body-cooler-cache:R R9
+L body-cooler:R R9
 U 1 1 5F0000A2
 P 7000 9800
@@
 $EndComp
 $Comp
-L body-cooler-cache:R R10
+L body-cooler:R R10
 U 1 1 5F0000A9
 P 7000 10600
@@
 $EndComp
 $Comp
-L body-cooler-cache:FLOW-YF-S401 FS1
+L body-cooler:FLOW-YF-S401 FS1
 U 1 1 5F0000B0
 P 8900 9400
@@
 5.4 开关量（全部用 MCU 内部上拉：引脚 — 开关 — GND）
 $Comp
-L body-cooler-cache:SW-LEVER SW1
+L body-cooler:SW-LEVER SW1
 U 1 1 5F0000B7
 P 2100 12500
@@
 GND
 $Comp
-L body-cooler-cache:SW-NC SW2
+L body-cooler:SW-NC SW2
 U 1 1 5F0000BE
 P 5100 12500
@@
 GND
 $Comp
-L body-cooler-cache:SW-PUSH SW3
+L body-cooler:SW-PUSH SW3
 U 1 1 5F0000C5
 P 2100 14000
@@
 GND
 $Comp
-L body-cooler-cache:SW-PUSH SW4
+L body-cooler:SW-PUSH SW4
 U 1 1 5F0000CC
 P 5100 14000
@@
 GND
 $Comp
-L body-cooler-cache:CONN-2 J1
+L body-cooler:CONN-2 J1
 U 1 1 5F0000D3
 P 6300 13000
@@
 5.5 蜂鸣器（可选）
 $Comp
-L body-cooler-cache:BUZZER LS1
+L body-cooler:BUZZER LS1
 U 1 1 5F0000DA
 P 9200 12500
